Commit message: fixed friction, joints

File: test_bot/urdf/bot.urdf (robot description, URDF)
Before this commit: robot m2wr, 4 links, 4 joints
Links:
- removed link caster_link
- added link caster_link_1, mass 0.2; collision sphere radius=0.033; visual sphere radius=0.033
- added link caster_link_2, mass 0.2; collision sphere radius=0.033; visual sphere radius=0.033
- added link dummy_link_1, mass 0.001
- added link dummy_link_2, mass 0.001
Joints:
- removed joint caster_joint_1
- removed joint caster_joint_2
- added joint caster_joint_11: type revolute, parent link_chassis, child dummy_link_1, origin xyz=0.2 0 -0.0675 rpy=0 0 0, axis 0 0 1, limit effort=0.26 velocity=20
- added joint caster_joint_12: type revolute, parent dummy_link_1, child caster_link_1, origin xyz=0 0 0 rpy=0 0 0, axis 0 1 0, limit effort=0.26 velocity=20
- added joint caster_joint_21: type revolute, parent link_chassis, child dummy_link_2, origin xyz=-0.2 0 -0.0675 rpy=0 0 0, axis 0 0 1, limit effort=0.26 velocity=20
- added joint caster_joint_22: type revolute, parent dummy_link_2, child caster_link_2, origin xyz=0 0 0 rpy=0 0 0, axis 0 1 0, limit effort=0.26 velocity=20
- joint joint_left_wheel: limit effort=0.26 velocity=20 -> effort=2.6 velocity=20; origin xyz=-0.05 -0.33 0 rpy=0 0 0 -> xyz=0 -0.33 0 rpy=0 0 0
- joint joint_right_wheel: limit effort=0.26 velocity=20 -> effort=2.6 velocity=20; origin xyz=-0.05 0.33 0 rpy=0 0 0 -> xyz=0 0.33 0 rpy=0 0 0
