Commit message: Changed xacro macro for scale in urdf

File: dot_description/urdf/bot.urdf.xacro (robot description, xacro)
@@ -1,4 +1,5 @@
 <?xml version="1.0" ?>
 <robot name="dot" xmlns:xacro="https://www.ros.org/wiki/xacro" >
+  <xacro:property name="scale" default="0.5" />
   <gazebo>
     <plugin name="gazebo_ros_control" filename="libgazebo_ros_control.so">
@@ -46,5 +47,5 @@
     <pose>0 0 0.1 0 0 0</pose>
     <inertial>
-      <mass value="5"/>
+      <mass value="${5 * scale}"/>
       <origin rpy="0 0 0" xyz="0 0 0"/>
       <inertia ixx="0.0395416666667" ixy="0" ixz="0" iyy="0.106208333333" iyz="0" izz="0.106208333333"/>
@@ -52,5 +53,5 @@
     <collision name="collision_chassis">
       <geometry>
-        <cylinder length="0.07" radius="0.3"/>
+        <cylinder length="${0.07 * scale}" radius="${0.3 * scale}"/>
       </geometry>
     </collision>
@@ -58,5 +59,5 @@
       <origin rpy="0 0 0" xyz="0 0 0"/>
       <geometry>
-        <cylinder length="0.07" radius="0.3"/>
+        <cylinder length="${0.07 * scale}" radius="${0.3 * scale}"/>
       </geometry>
       <material name="red"/>
@@ -66,5 +67,5 @@
   <link name="caster_link_1">
     <inertial>
-      <mass value="0.2"/>
+      <mass value="${0.2 * scale}"/>
       <origin rpy="0 0 0" xyz="0 0 0"/>
       <inertia ixx="0.00052666666" ixy="0" ixz="0" iyy="0.00052666666" iyz="0" izz="0.001"/>
@@ -73,5 +74,5 @@
       <origin rpy="0 0 0" xyz="0 0 0" />
       <geometry>
-        <sphere radius="0.033"/>
+        <sphere radius="${0.033 * scale}"/>
       </geometry>
     </collision>
@@ -79,5 +80,5 @@
       <origin rpy="0 0 0" xyz="0 0 0"/>
       <geometry>
-        <sphere radius="0.033"/>
+        <sphere radius="${0.033 * scale}"/>
       </geometry>
     </visual>
@@ -85,5 +86,5 @@
   <link name="dummy_link_1">
     <inertial>
-      <mass value="0.001"/>
+      <mass value="${0.001 * scale}"/>
       <origin rpy="0 0 0" xyz="0 0 0"/>
       <inertia ixx="0" ixy="0" ixz="0" iyy="0.0" iyz="0" izz="0"/>
@@ -91,5 +92,5 @@
   </link>
   <joint name="caster_joint_11" type="revolute">
-    <origin rpy="0 0 0" xyz="0.2 0 -0.0675" />
+    <origin rpy="0 0 0" xyz="${0.2 * scale} ${0 * scale} ${-0.0675 * scale}" />
     <child link="dummy_link_1" />
     <parent link="link_chassis" />
@@ -108,5 +109,5 @@
   <link name="caster_link_2">
     <inertial>
-      <mass value="0.2"/>
+      <mass value="${0.2 * scale}"/>
       <origin rpy="0 0 0" xyz="0 0 0"/>
       <inertia ixx="0.00052666666" ixy="0" ixz="0" iyy="0.00052666666" iyz="0" izz="0.001"/>
@@ -115,5 +116,5 @@
       <origin rpy="0 0 0" xyz="0 0 0" />
       <geometry>
-        <sphere radius="0.033"/>
+        <sphere radius="${0.033 * scale}"/>
       </geometry>
     </collision>
@@ -121,5 +122,5 @@
       <origin rpy="0 0 0" xyz="0 0 0"/>
       <geometry>
-        <sphere radius="0.033"/>
+        <sphere radius="${0.033 * scale}"/>
       </geometry>
     </visual>
@@ -127,5 +128,5 @@
   <link name="dummy_link_2">
     <inertial>
-      <mass value="0.001"/>
+      <mass value="${0.001 * scale}"/>
       <origin rpy="0 0 0" xyz="0 0 0"/>
       <inertia ixx="0" ixy="0" ixz="0" iyy="0.0" iyz="0" izz="0"/>
@@ -133,5 +134,5 @@
   </link>
   <joint name="caster_joint_21" type="revolute">
-    <origin rpy="0 0 0" xyz="-0.2 0 -0.0675"/>
+    <origin rpy="0 0 0" xyz="${-0.2 * scale} ${0 * scale} ${-0.0675 * scale}"/>
     <child link="dummy_link_2" />
     <parent link="link_chassis" />
@@ -151,5 +152,5 @@
   <link name="link_right_wheel">
     <inertial>
-      <mass value="0.2"/>
+      <mass value="${0.2 * scale}"/>
       <origin rpy="0 1.5707 1.5707" xyz="0 0 0"/>
       <inertia ixx="0.00052666666" ixy="0" ixz="0" iyy="0.00052666666" iyz="0" izz="0.001"/>
@@ -158,5 +159,5 @@
       <origin rpy="0 1.5707 1.5707" xyz="0 0 0" />
       <geometry>
-        <cylinder length="0.04" radius="0.1"/>
+        <cylinder length="${0.04 * scale}" radius="${0.1 * scale}"/>
       </geometry>
     </collision>
@@ -164,5 +165,5 @@
       <origin rpy="0 1.5707 1.5707" xyz="0 0 0"/>
       <geometry>
-        <cylinder length="0.04" radius="0.1"/>
+        <cylinder length="${0.04 * scale}" radius="${0.1 * scale}"/>
       </geometry>
     </visual>
@@ -170,8 +171,8 @@
   <!--   Joint for right wheel  -->
   <joint name="joint_right_wheel" type="continuous">
-    <origin rpy="0 0 0" xyz="0 0.33 0"/>
+    <origin rpy="0 0 0" xyz="${0 * scale} ${0.33 * scale} ${0 * scale}"/>
     <child link="link_right_wheel" />
     <parent link="link_chassis"/>
-    <axis rpy="0 0 0" xyz="0 1 0"/>
+    <axis rpy="0 0 0" xyz="${0 * scale} ${1 * scale} ${0 * scale}"/>
     <limit effort="2.6" velocity="20"/>
     <joint_properties damping="0.1" friction="0.1" />
@@ -180,5 +181,5 @@
   <link name="link_left_wheel">
     <inertial>
-      <mass value="0.2"/>
+      <mass value="${0.2 * scale}"/>
       <origin rpy="0 1.5707 1.5707" xyz="0 0 0"/>
       <inertia ixx="0.00052666666" ixy="0" ixz="0" iyy="0.00052666666" iyz="0" izz="0.001"/>
@@ -187,5 +188,5 @@
       <origin rpy="0 1.5707 1.5707" xyz="0 0 0" />
       <geometry>
-        <cylinder length="0.04" radius="0.1"/>
+        <cylinder length="${0.04 * scale}" radius="${0.1 * scale}"/>
       </geometry>
     </collision>
@@ -193,5 +194,5 @@
       <origin rpy="0 1.5707 1.5707" xyz="0 0 0"/>
       <geometry>
-        <cylinder length="0.04" radius="0.1"/>
+        <cylinder length="${0.04 * scale}" radius="${0.1 * scale}"/>
       </geometry>
     </visual>
@@ -199,5 +200,5 @@
   <!--   Joint for left wheel  -->
   <joint name="joint_left_wheel" type="continuous">
-    <origin rpy="0 0 0" xyz="0 -0.33 0"/>
+    <origin rpy="0 0 0" xyz="${0 * scale} ${-0.33 * scale} ${0 * scale}"/>
     <child link="link_left_wheel" />
     <parent link="link_chassis"/>

Commit message: ..

File: dot_description/urdf/bot.urdf.xacro (robot description, xacro)
@@ -2,4 +2,5 @@
 <robot name="dot" xmlns:xacro="https://www.ros.org/wiki/xacro" >
   <xacro:property name="scale" default="0.5" />
+  <xacro:property name="camera_link" value="0.05" /> <!-- Size of square 'camera' box -->
   <gazebo>
     <plugin name="gazebo_ros_control" filename="libgazebo_ros_control.so">
@@ -227,3 +228,66 @@
     </actuator>
   </transmission>
+  <!-- Block Laser -->
+  <joint name="hokuyo_joint" type="fixed">
+    <axis xyz="0 1 0" />
+    <origin xyz="${camera_link} 0 0.05" rpy="0 0 0"/>
+    <parent link="link_chassis"/>
+    <child link="hokuyo_link"/>
+  </joint>
+  <!-- Hokuyo Laser -->
+  <link name="hokuyo_link">
+    <collision>
+      <origin xyz="0 0 0" rpy="0 0 0"/>
+      <geometry>
+    <box size="0.1 0.1 0.1"/>
+      </geometry>
+    </collision>
+    <visual>
+      <origin xyz="0 0 0" rpy="0 0 0"/>
+      <geometry>
+        <box size="${camera_link} ${camera_link} ${camera_link}"/>
+      </geometry>
+    </visual>
+    <inertial>
+      <mass value="1e-5" />
+      <origin xyz="0 0 0" rpy="0 0 0"/>
+      <inertia ixx="1e-6" ixy="0" ixz="0" iyy="1e-6" iyz="0" izz="1e-6" />
+    </inertial>
+  </link>
+  <!-- hokuyo -->
+  <gazebo reference="hokuyo_link">
+    <sensor type="gpu_ray" name="head_hokuyo_sensor">
+      <pose>0 0 0 0 0 0</pose>
+      <visualize>false</visualize>
+      <update_rate>40</update_rate>
+      <ray>
+        <scan>
+          <horizontal>
+            <samples>720</samples>
+            <resolution>1</resolution>
+            <min_angle>-1.570796</min_angle>
+            <max_angle>1.570796</max_angle>
+          </horizontal>
+        </scan>
+        <range>
+          <min>0.10</min>
+          <max>30.0</max>
+          <resolution>0.01</resolution>
+        </range>
+        <noise>
+          <type>gaussian</type>
+          <!-- Noise parameters based on published spec for Hokuyo laser
+               achieving "+-30mm" accuracy at range < 10m.  A mean of 0.0m and
+               stddev of 0.01m will put 99.7% of samples within 0.03m of the true
+               reading. -->
+          <mean>0.0</mean>
+          <stddev>0.01</stddev>
+        </noise>
+      </ray>
+      <plugin name="gazebo_ros_head_hokuyo_controller" filename="libgazebo_ros_gpu_laser.so">
+        <topicName>/dot/laser/scan</topicName>
+        <frameName>hokuyo_link</frameName>
+      </plugin>
+    </sensor>
+  </gazebo>
 </robot>

Commit message: Added IMU sensor

File: dot_description/urdf/bot.urdf.xacro (robot description, xacro)
@@ -231,5 +231,5 @@
   <joint name="hokuyo_joint" type="fixed">
     <axis xyz="0 1 0" />
-    <origin xyz="${camera_link} 0 0.05" rpy="0 0 0"/>
+    <origin xyz="${camera_link} 0 ${0.07 * scale}" rpy="0 0 0"/>
     <parent link="link_chassis"/>
     <child link="hokuyo_link"/>
@@ -259,5 +259,5 @@
     <sensor type="gpu_ray" name="head_hokuyo_sensor">
       <pose>0 0 0 0 0 0</pose>
-      <visualize>false</visualize>
+      <visualize>true</visualize>
       <update_rate>40</update_rate>
       <ray>

File: dot_description/xacro/main.urdf.xacro (robot description, xacro)
@@ -60,4 +60,114 @@
 		rpy="1.570796326794896 0 -1.047197551196597"
 	/>
+	<!-- Block Laser -->
+  <joint name="hokuyo_joint" type="fixed">
+    <axis xyz="0 1 0" />
+    <origin xyz="0 0 0.01905" rpy="0 0 0"/>
+    <parent link="base_link"/>
+    <child link="hokuyo_link"/>
+  </joint>
+  <!-- Hokuyo Laser -->
+  <link name="hokuyo_link">
+    <collision>
+      <origin xyz="0 0 0" rpy="0 0 0"/>
+      <geometry>
+    <box size="0.01 0.01 0.01"/>
+      </geometry>
+    </collision>
+    <visual>
+      <origin xyz="0 0 0" rpy="0 0 0"/>
+      <geometry>
+        <box size="0.01 0.01 0.01"/>
+      </geometry>
+    </visual>
+    <inertial>
+      <mass value="1e-5" />
+      <origin xyz="0 0 0" rpy="0 0 0"/>
+      <inertia ixx="1e-6" ixy="0" ixz="0" iyy="1e-6" iyz="0" izz="1e-6" />
+    </inertial>
+  </link>
+  <!-- hokuyo -->
+  <gazebo reference="hokuyo_link">
+    <sensor type="ray" name="head_hokuyo_sensor">
+      <pose>0 0 0 0 0 0</pose>
+      <visualize>false</visualize>
+      <update_rate>40</update_rate>
+      <ray>
+        <scan>
+          <horizontal>
+            <samples>720</samples>
+            <resolution>1</resolution>
+            <min_angle>-1.570796</min_angle>
+            <max_angle>1.570796</max_angle>
+          </horizontal>
+        </scan>
+        <range>
+          <min>0.1</min>
+          <max>30</max>
+          <resolution>0.01</resolution>
+        </range>
+        <noise>
+          <type>gaussian</type>
+          <!-- Noise parameters based on published spec for Hokuyo laser
+               achieving "+-30mm" accuracy at range < 10m.  A mean of 0.0m and
+               stddev of 0.01m will put 99.7% of samples within 0.03m of the true
+               reading. -->
+          <mean>0.0</mean>
+          <stddev>0.01</stddev>
+        </noise>
+      </ray>
+      <plugin filename="libgazebo_ros_laser.so" name="gazebo_ros_head_hokuyo_controller">
+        <topicName>/dot/laser_scan</topicName>
+        <frameName>hokuyo_link</frameName>
+      </plugin>
+    </sensor>
+  </gazebo>
+  <joint name="imu_joint" type="fixed">
+      <axis xyz="0 0 1" />
+      <origin xyz="0 0 0.015" rpy="0 0 0"/>
+      <parent link="base_link"/>
+      <child link="imu_link"/>
+  </joint>
+  <!-- Imu Link-->
+  <link name="imu_link">
+        <collision>
+            <origin xyz="0 0 0" rpy="0 0 0"/>
+            <geometry>
+                <box size="0.01 0.01 0.01"/>
+            </geometry>
+        </collision>
+        <visual>
+            <origin xyz="0 0 0" rpy="0 0 0"/>
+            <geometry>
+                <box size="0.01 0.01 0.01"/>
+            </geometry>
+        </visual>
+        <inertial>
+            <mass value="0.001" />
+            <origin xyz="0 0 0" rpy="0 0 0"/>
+            <inertia ixx="0.00000015" ixy="0" ixz="0" iyy="0.00000015" iyz="0" izz="0.00000015" />
+        </inertial>
+  </link>
+  <!--IMU Link gazebo plugin-->
+  <gazebo reference="imu_link">
+    <gravity>true</gravity>
+    <sensor name="imu_sensor" type="imu">
+      <always_on>true</always_on>
+      <update_rate>100</update_rate>
+      <visualize>true</visualize>
+      <topic>__default_topic__</topic>
+      <plugin filename="libgazebo_ros_imu_sensor.so" name="imu_plugin">
+        <topicName>/dot/imu</topicName>
+        <bodyName>imu_link</bodyName>
+        <updateRateHZ>10.0</updateRateHZ>
+        <gaussianNoise>0.0</gaussianNoise>
+        <xyzOffset>0 0 0</xyzOffset>
+        <rpyOffset>0 0 0</rpyOffset>
+        <frameName>imu_link</frameName>
+        <initialOrientationAsReference>false</initialOrientationAsReference>
+      </plugin>
+      <pose>0 0 0 0 0 0</pose>
+    </sensor>
+  </gazebo>
 	<gazebo>
 		<plugin name="gazebo_ros_control" filename="libgazebo_ros_control.so">
