Commit message: updated urdf

File: dot_description/xacro/main.urdf.xacro (robot description, xacro)
@@ -42,5 +42,5 @@
 		/>
 	</joint>
-	<xacro:rim_macro
+	<!-- <xacro:rim_macro
 		name="left"
 		color="0.3 0 0"
@@ -58,4 +58,22 @@
 		color="0 0 0.3"
 		xyz="0.03464101615 0.02 0"
+		rpy="1.570796326794896 0 -1.047197551196597"
+	/> -->
+	<xacro:rim_macro
+		name="left"
+		color="0.3 0 0"
+		xyz="0.0407838 -0.0190178218 -0.025"
+		rpy="1.570796326794896 0 1.047197551196597"
+	/>
+	<xacro:rim_macro
+		name="back"
+		color="0 0.3 0"
+		xyz="-0.001 0.041 -0.025"
+		rpy="1.570796326794896 0 3.141592653589793"
+	/>
+	<xacro:rim_macro
+		name="right"
+		color="0 0 0.3"
+		xyz="-0.03464101615 -0.02 -0.025"
 		rpy="1.570796326794896 0 -1.047197551196597"
 	/>
@@ -65,3 +83,171 @@
 		</plugin>
 	</gazebo>
+	<joint name="dummy_joint" type="fixed">
+    <parent link="base_link"/>
+    <child link="platform_base"/>
+	<origin rpy="0 0 0" xyz="0 0 0.028" />
+</joint>
+<link name='platform_base'>
+    <inertial>
+        <origin rpy="0 0 0" xyz="0 0 0"/>
+        <mass value="0.2"/>
+        <inertia ixx="0.06" ixy="0" ixz="0" iyy="0.06" iyz="0" izz="0.12"/>
+    </inertial>
+    <visual>
+        <material name="Cyan">
+            <color rgba="0 1.0 1.0 1.0" />
+        </material>
+        <origin rpy="0 0 0" xyz="0 0 0"/>
+        <geometry>
+            <box size="0.092 0.092 0.002"/>
+        </geometry>
+    </visual>
+    <collision>
+        <origin rpy="0 0 0" xyz="0 0 0"/>
+        <geometry>
+            <box size="0.092 0.092 0.002"/>
+        </geometry>
+    </collision>
+</link>
+<gazebo reference="platform_base">
+    <material>Gazebo/Black</material>
+    <kp>10000000.0</kp>
+    <kd>1.0</kd>
+    <mu1>4.0</mu1>
+    <mu2>4.0</mu2>
+    <maxVel>0.0</maxVel>
+    <minDepth>0.001</minDepth>
+</gazebo>
+<joint name="dummy_base" type="fixed">
+    <origin rpy="0 0 0" xyz="0 0 0.013" />
+    <parent link="platform_base"/>
+    <child link="ball"/>
+</joint>
+<link name='ball'>
+    <inertial>
+        <origin rpy="0 0 0" xyz="0 0 0"/>
+        <mass value="0.5"/>
+        <inertia ixx="0.1" ixy="0" ixz="0" iyy="0.1" iyz="0" izz="0.1"/>
+    </inertial>
+    <visual>
+        <origin rpy="0 0 0" xyz="0 0 0"/>
+        <geometry>
+            <sphere radius="0.013"/>
+        </geometry>
+        <material name="gray">
+            <color rgba="0.7 0.7 0.7 1"/>
+        </material>
+    </visual>
+    <collision>
+        <origin rpy="0 0 0" xyz="0 0 0"/>
+        <geometry>
+            <sphere radius="0.013"/>
+        </geometry>
+    </collision>
+</link>
+<gazebo reference="ball">
+    <material>Gazebo/DarkGrey</material>
+    <kp>10000000.0</kp>
+    <kd>1.0</kd>
+    <mu1>4.0</mu1>
+    <mu2>4.0</mu2>
+    <maxVel>0.0</maxVel>
+    <minDepth>0.001</minDepth>
+</gazebo>
+<link name='platform'>
+    <inertial>
+        <origin rpy="0 0 0" xyz="0 0 0"/>
+        <mass value="0.2"/>
+        <inertia ixx="0.06" ixy="0" ixz="0" iyy="0.06" iyz="0" izz="0.12"/>
+    </inertial>
+    <visual>
+        <material name="Cyan">
+            <color rgba="0 1.0 1.0 1.0" />
+        </material>
+        <origin rpy="0 0 0" xyz="0 0 0"/>
+        <geometry>
+            <box size="0.092 0.092 0.002"/>
+        </geometry>
+    </visual>
+    <collision>
+        <origin rpy="0 0 0" xyz="0 0 0"/>
+        <geometry>
+            <box size="0.092 0.092 0.0015"/>
+        </geometry>
+    </collision>
+</link>
+<gazebo reference="platform">
+    <material>Gazebo/Orange</material>
+    <kp>10000000.0</kp>
+    <kd>1.0</kd>
+    <mu1>4.0</mu1>
+    <mu2>4.0</mu2>
+    <maxVel>0.0</maxVel>
+    <minDepth>0.001</minDepth>
+</gazebo>
+<link name='platform_mid'>
+    <inertial>
+        <origin rpy="1.57 0 0" xyz="0 0 0"/>
+        <mass value="0.1"/>
+        <inertia ixx="0.01" ixy="0" ixz="0" iyy="0.01" iyz="0" izz="0.12"/>
+    </inertial>
+    <visual>
+        <material name="black">
+            <color rgba="0 0 0 1.0" />
+        </material>
+        <origin rpy="1.57 0 0" xyz="0 0 0"/>
+        <geometry>
+            <cylinder radius="0.001" length="0.002" />
+        </geometry>
+    </visual>
+    <collision>
+        <origin rpy="1.57 0 0" xyz="0 0 0"/>
+        <geometry>
+            <cylinder radius="0.001" length="0.002" />
+        </geometry>
+    </collision>
+</link>
+<gazebo reference="platform_mid">
+    <material>Gazebo/White</material>
+    <kp>10000000.0</kp>
+    <kd>1.0</kd>
+    <mu1>4.0</mu1>
+    <mu2>4.0</mu2>
+    <maxVel>0.0</maxVel>
+    <minDepth>0.001</minDepth>
+</gazebo>
+<joint name='rev_x' type='revolute'>
+    <origin rpy="0.0 0.0 0.0" xyz="0.0 0.0 0.014"/>
+    <parent link="ball"/>
+    <child link="platform_mid"/>
+    <axis xyz="1 0 0"/>
+    <limit lower="-0.05" upper="0.05" effort="2e+2" velocity="1" />
+</joint>
+<joint name='rev_y' type='revolute'>
+    <origin rpy="0.0 0.0 0.0" xyz="0.0 0.0 0.001"/>
+    <parent link="platform_mid"/>
+    <child link="platform"/>
+    <axis xyz="0 1 0"/>
+    <limit lower="-0.05" upper="0.05" effort="2e+2" velocity="1" />
+</joint>
+<transmission name="simple_trans1">
+    <type>transmission_interface/SimpleTransmission</type>
+    <joint name="rev_x">
+    <hardwareInterface>hardware_interface/EffortJointInterface</hardwareInterface>
+    </joint>
+    <actuator name="motor_x">
+    <mechanicalReducation>50</mechanicalReducation>
+    <hardwareInterface>hardware_interface/EffortJointInterface</hardwareInterface>
+    </actuator>
+</transmission>
+<transmission name="simple_trans2">
+    <type>transmission_interface/SimpleTransmission</type>
+    <joint name="rev_y">
+    <hardwareInterface>hardware_interface/EffortJointInterface</hardwareInterface>
+    </joint>
+    <actuator name="motor_y">
+    <mechanicalReducation>50</mechanicalReducation>
+    <hardwareInterface>hardware_interface/EffortJointInterface</hardwareInterface>
+    </actuator>
+</transmission>
 </robot>

Commit message: urdf updated

File: dot_description/xacro/main.urdf.xacro (robot description, xacro)
@@ -42,5 +42,5 @@
 		/>
 	</joint>
-	<!-- <xacro:rim_macro
+	<xacro:rim_macro
 		name="left"
 		color="0.3 0 0"
@@ -59,9 +59,9 @@
 		xyz="0.03464101615 0.02 0"
 		rpy="1.570796326794896 0 -1.047197551196597"
-	/> -->
-	<xacro:rim_macro
+	/>
+	<!-- <xacro:rim_macro
 		name="left"
 		color="0.3 0 0"
-		xyz="0.0407838 -0.0190178218 -0.025"
+		xyz="0.0453153894 -0.021139091 -0.025"
 		rpy="1.570796326794896 0 1.047197551196597"
 	/>
@@ -69,5 +69,5 @@
 		name="back"
 		color="0 0.3 0"
-		xyz="-0.001 0.041 -0.025"
+		xyz="-0.001 0.046 -0.025"
 		rpy="1.570796326794896 0 3.141592653589793"
 	/>
@@ -75,7 +75,7 @@
 		name="right"
 		color="0 0 0.3"
-		xyz="-0.03464101615 -0.02 -0.025"
+		xyz="-0.0433012702 -0.025 -0.025"
 		rpy="1.570796326794896 0 -1.047197551196597"
-	/>
+	/> -->
 	<gazebo>
 		<plugin name="gazebo_ros_control" filename="libgazebo_ros_control.so">
@@ -83,14 +83,138 @@
 		</plugin>
 	</gazebo>
-	<joint name="dummy_joint" type="fixed">
+<link name="supp_cyl">
+	<!-- <inertial>
+		<mass value="0.04"/>
+		<inertia
+			ixx="2.08e-06"
+			ixy="0"
+			ixz="0"
+			iyy="2.08e-06"
+			iyz="0"
+			izz="1.67e-09"
+		/>
+	</inertial> -->
+	<visual>
+		<geometry>
+			<cylinder radius="0.001" length="0.025"/>
+		</geometry>
+		<material name="base_material">
+			<color rgba="1 1 1 1"/>
+		</material>
+	</visual>
+	<collision>
+		<geometry>
+			<cylinder radius="0.001" length="0.025"/>
+		</geometry>
+	</collision>
+	</link>
+<link name="mid_cyl">
+	<!-- <inertial>
+		<mass value="0.07862944645"/>
+		<inertia
+			ixx="0.00002035985530754"
+			ixy="0"
+			ixz="0"
+			iyy="0.00002035985530754"
+			iyz="0"
+			izz="0.00003945961663220"
+		/>
+	</inertial> -->
+	<visual>
+		<geometry>
+			<cylinder radius="0.04" length="0.001"/>
+		</geometry>
+		<material name="base_material">
+			<color rgba="1 1 1 1"/>
+		</material>
+	</visual>
+	<collision>
+		<geometry>
+			<cylinder radius="0.04" length="0.001"/>
+		</geometry>
+	</collision>
+	</link>
+<joint name="supp_mid" type="fixed">
+    <origin xyz="0 0 0.0125" rpy="0 0 0"/>
+    <parent link="supp_cyl"/>
+    <child link="mid_cyl"/>
+ </joint>
+ <joint name="supp_base" type="fixed">
+    <origin xyz="0 0 0.0125" rpy="0 0 0"/>
     <parent link="base_link"/>
+    <child link="supp_cyl"/>
+</joint>
+	<link name="supp_cyl_2">
+	<!-- <inertial>
+		<mass value="0.04"/>
+		<inertia
+			ixx="2.08e-06"
+			ixy="0"
+			ixz="0"
+			iyy="2.08e-06"
+			iyz="0"
+			izz="1.67e-09"
+		/>
+	</inertial> -->
+	<visual>
+		<geometry>
+			<cylinder radius="0.001" length="0.025"/>
+		</geometry>
+		<material name="base_material">
+			<color rgba="1 1 1 1"/>
+		</material>
+	</visual>
+	<collision>
+		<geometry>
+			<cylinder radius="0.001" length="0.025"/>
+		</geometry>
+	</collision>
+	</link>
+<link name="mid_cyl_2">
+	<!-- <inertial>
+		<mass value="0.07862944645"/>
+		<inertia
+			ixx="0.00002035985530754"
+			ixy="0"
+			ixz="0"
+			iyy="0.00002035985530754"
+			iyz="0"
+			izz="0.00003945961663220"
+		/>
+	</inertial> -->
+	<visual>
+		<geometry>
+			<cylinder radius="0.04" length="0.001"/>
+		</geometry>
+		<material name="base_material">
+			<color rgba="1 1 1 1"/>
+		</material>
+	</visual>
+	<collision>
+		<geometry>
+			<cylinder radius="0.04" length="0.001"/>
+		</geometry>
+	</collision>
+	</link>
+<joint name="supp_mid_2" type="fixed">
+    <origin xyz="0 0 0.0125" rpy="0 0 0"/>
+    <parent link="supp_cyl_2"/>
+    <child link="mid_cyl_2"/>
+ </joint>
+ <joint name="supp_base_2" type="fixed">
+    <origin xyz="0 0 0.0125" rpy="0 0 0"/>
+    <parent link="mid_cyl"/>
+    <child link="supp_cyl_2"/>
+ </joint>
+ <joint name="dummy_joint" type="fixed">
+    <parent link="mid_cyl_2"/>
     <child link="platform_base"/>
-	<origin rpy="0 0 0" xyz="0 0 0.028" />
+	<origin rpy="0 0 0" xyz="0 0 0.001" />
 </joint>
 <link name='platform_base'>
     <inertial>
         <origin rpy="0 0 0" xyz="0 0 0"/>
-        <mass value="0.2"/>
-        <inertia ixx="0.06" ixy="0" ixz="0" iyy="0.06" iyz="0" izz="0.12"/>
+        <mass value="0.002"/>
+        <inertia ixx="0.0006" ixy="0" ixz="0" iyy="0.0006" iyz="0" izz="0.0012"/>
     </inertial>
     <visual>
@@ -127,6 +251,6 @@
     <inertial>
         <origin rpy="0 0 0" xyz="0 0 0"/>
-        <mass value="0.5"/>
-        <inertia ixx="0.1" ixy="0" ixz="0" iyy="0.1" iyz="0" izz="0.1"/>
+        <mass value="0.005"/>
+        <inertia ixx="0.001" ixy="0" ixz="0" iyy="0.001" iyz="0" izz="0.001"/>
     </inertial>
     <visual>
@@ -158,6 +282,6 @@
     <inertial>
         <origin rpy="0 0 0" xyz="0 0 0"/>
-        <mass value="0.2"/>
-        <inertia ixx="0.06" ixy="0" ixz="0" iyy="0.06" iyz="0" izz="0.12"/>
+        <mass value="0.002"/>
+        <inertia ixx="0.0006" ixy="0" ixz="0" iyy="0.0006" iyz="0" izz="0.0012"/>
     </inertial>
     <visual>
@@ -189,6 +313,6 @@
     <inertial>
         <origin rpy="1.57 0 0" xyz="0 0 0"/>
-        <mass value="0.1"/>
-        <inertia ixx="0.01" ixy="0" ixz="0" iyy="0.01" iyz="0" izz="0.12"/>
+        <mass value="0.001"/>
+        <inertia ixx="0.0001" ixy="0" ixz="0" iyy="0.0001" iyz="0" izz="0.0012"/>
     </inertial>
     <visual>

Commit message: Adding camera,tracking_pid

File: dot_description/xacro/main.urdf.xacro (robot description, xacro)
@@ -389,4 +389,54 @@
     <minDepth>0.001</minDepth>
 </gazebo>
+<link name='platform_tag0'>
+    <inertial>
+        <origin rpy="0 0 0" xyz="0 0 0"/>
+        <mass value="0.002"/>
+        <inertia ixx="0.0006" ixy="0" ixz="0" iyy="0.0006" iyz="0" izz="0.0012"/>
+    </inertial>
+    <visual>
+        <material name="Cyan">
+            <color rgba="0 1.0 1.0 1.0" />
+        </material>
+        <origin rpy="0 0 0" xyz="0 0 0"/>
+        <geometry>
+            <mesh filename="package://dot_description/mesh/tag0/tag0.dae" scale="0.45 0.45 1"/>
+        </geometry>
+    </visual>
+</link>
+<gazebo reference="platform_tag1">
+    <material>package://dot_description/mesh/tag0/gazebo.material</material>
+    <kp>10000000.0</kp>
+    <kd>1.0</kd>
+    <mu1>4.0</mu1>
+    <mu2>4.0</mu2>
+    <maxVel>0.0</maxVel>
+    <minDepth>0.001</minDepth>
+</gazebo>
+<link name='platform_tag1'>
+    <inertial>
+        <origin rpy="0 0 0" xyz="0 0 0"/>
+        <mass value="0.002"/>
+        <inertia ixx="0.0006" ixy="0" ixz="0" iyy="0.0006" iyz="0" izz="0.0012"/>
+    </inertial>
+    <visual>
+        <material name="Cyan">
+            <color rgba="0 1.0 1.0 1.0" />
+        </material>
+        <origin rpy="0 0 0" xyz="0 0 0"/>
+        <geometry>
+            <mesh filename="package://dot_description/mesh/tag1/tag1.dae" scale="0.45 0.45 1"/>
+        </geometry>
+    </visual>
+</link>
+<gazebo reference="platform_tag1">
+    <material>package://dot_description/mesh/tag1/gazebo.material</material>
+    <kp>10000000.0</kp>
+    <kd>1.0</kd>
+    <mu1>4.0</mu1>
+    <mu2>4.0</mu2>
+    <maxVel>0.0</maxVel>
+    <minDepth>0.001</minDepth>
+</gazebo>
 <link name='platform'>
     <inertial>
@@ -464,4 +514,14 @@
     <axis xyz="0 1 0"/>
     <limit lower="-0.05" upper="0.05" effort="2e+2" velocity="1" />
+</joint>
+<joint name='fixed_joint0' type='fixed'>
+    <origin rpy="0.0 0.0 0.0" xyz="-0.023 -0.023 0.008"/>
+    <parent link="platform_mid"/>
+    <child link="platform_tag0"/>
+</joint>
+<joint name='fixed_joint1' type='fixed'>
+    <origin rpy="0.0 0.0 0.0" xyz="0.023 0.023 0.008"/>
+    <parent link="platform_mid"/>
+    <child link="platform_tag1"/>
 </joint>
 <transmission name="simple_trans1">

File: dot_gazebo/urdf/cameras.urdf (robot description, URDF)
Before this commit: robot bot, 5 links, 4 joints
Links:
- added link april1, mass 0.002; visual mesh filename=package://dot_description/mesh/tag13/tag13.dae scale=1 1 1
- added link april2, mass 0.002; visual mesh filename=package://dot_description/mesh/tag14/tag14.dae scale=1 1 1
- added link april3, mass 0.002; visual mesh filename=package://dot_description/mesh/tag15/tag15.dae scale=1 1 1
Joints:
- added joint apri1: type fixed, parent world, child april1, origin xyz=0 0 0.04 rpy=0 0 0
- added joint apri2: type fixed, parent world, child april2, origin xyz=0.6096 0 0.04 rpy=0 0 0
- added joint apri3: type fixed, parent world, child april3, origin xyz=-0.6096 0 0.04 rpy=0 0 0
